Commit message: added hand continuous joint/link

File: scara_52900/urdf/scara_arm_pvc.urdf (robot description, URDF)
Before this commit: robot scara_arm_pvc, 5 links, 4 joints
Links:
- link hand: geometry visual box size=.03 .129 .009
Joints:
- joint elbow: origin xyz=0 .190 -.08 rpy=0 0 0 -> xyz=0 .190 -.065 rpy=0 0 0
- joint wrist: origin xyz=52 0 27 rpy=0 0 0 -> xyz=0 .1993 -.05 rpy=1.57057 0  0 

Commit message: before http://wiki.ros.org/urdf/Tutorials/Using%20a%20URDF%20in%20Gazebo tutorial

File: scara_52900/urdf/scara_arm_pvc.urdf (robot description, URDF)
Before this commit: robot scara_arm_pvc, 5 links, 4 joints
Links:
- link base_link: geometry collision box size=.139 .195 .009; visual box size=.139 .195 .009
- link forearm: geometry collision box size=.205 .06 .072; visual box size=.205 .06 .072
- link hand: geometry collision box size=.03 .129 .009; visual box size=.03 .129 .009
- link humerus: geometry collision box size=.255 .059 .056; visual box size=.255 .059 .056
- link scapula: geometry collision box size=.155 .134 .320; visual box size=.155 .134 .320
Joints:
- joint shoulder: origin xyz=0 0 0 rpy=0 0 0 -> xyz=0 0 .04 rpy=0 0 0
- joint waist: limit lower=0 upper=6 effort=1 velocity=1 -> lower=-3 upper=3 effort=1 velocity=1
