Commit message: updated joint locations

File: urdf/scara_52900.urdf.xacro (robot description, xacro)
@@ -34,4 +34,5 @@
       </geometry>
       <material name="pvc"/>
+      <origin rpy="0 0 0" xyz="0 0 0" />
     </visual>
     <collision>
@@ -42,7 +43,15 @@
     <inertial>
     	<mass value="4" />
-    <inertia ixx="0.4" ixy="0.0" ixz="0.0" iyy="0.4" iyz="0.0" izz="0.2"/>
+      <inertia ixx="1e-3" ixy="0.0" ixz="0.0" iyy="1e-3" iyz="0.0" izz="1e-3"/>
+      <origin xyz="0 0 0" rpy="0 0 0" />
   	</inertial>
   </link>
+  <!-- Used for fixing robot to Gazebo 'base_link' -->
+  <link name="world"/>
+  <joint name="fixed" type="fixed">
+    <parent link="world"/>
+    <child link="base_link"/>
+    <origin xyz="0 0 0"/>
+  </joint>
   <link name="scapula">
     <visual>
@@ -86,7 +95,7 @@
     <visual>
       <geometry>
-        <box size=".255 .059 .056"/>
-      </geometry>
-      <origin rpy="0 0 1.57057" xyz="0 .110 0"/>
+        <box size=".200 .059 .056"/>
+      </geometry>
+      <origin rpy="0 0 1.57057" xyz="0 .100 0"/>
       <material name="pvc"/>
     </visual>
@@ -121,18 +130,18 @@
     <visual>
       <geometry>
-        <box size=".205 .06 .072"/>
-      </geometry>
-      <origin xyz="0 .100 0" rpy="0 0 1.57057" />
+        <box size=".150 .06 .072"/>
+      </geometry>
+      <origin xyz="0 .0750 0" rpy="0 0 1.57057" />
       <material name="blue"/>
     </visual>
     <collision>
       <geometry>
-        <box size=".205 .06 .072"/>
-      </geometry>
-    </collision>
-    <inertial>
-    		<mass value="${mass_upper_links}" />
-    <inertia ixx="0.4" ixy="0.0" ixz="0.0" iyy="0.4" iyz="0.0" izz="0.2"/>
-  </inertial>
+        <box size=".150 .06 .072"/>
+      </geometry>
+    </collision>
+    <inertial>
+    	<mass value="${mass_upper_links}" />
+      <inertia ixx="0.4" ixy="0.0" ixz="0.0" iyy="0.4" iyz="0.0" izz="0.2"/>
+    </inertial>
   </link>
   <joint name="elbow" type="revolute">
@@ -140,5 +149,5 @@
     <child link="forearm"/>
     <limit lower="-2.44" upper="2.44" effort="30" velocity="1"/>
-    <origin xyz="0 .190 -.065" rpy="0 0 0" />
+    <origin xyz="0 .200 -.065" rpy="0 0 0" />
     <axis xyz="0 0 1" />
     <dynamics damping="${damping_value}" friction="${friction_value}" />
@@ -174,5 +183,5 @@
     <parent link="forearm"/>
     <child link="hand"/>
-    <origin xyz="0 .1993 -.05" rpy="1.57057 0  0 " />
+    <origin xyz="0 .150 -.05" rpy="1.57057 0  0 " />
     <axis xyz="0 1 0" />
     <dynamics damping="${damping_value}" friction="${friction_value}" />
@@ -193,3 +202,7 @@
     </plugin>
   </gazebo>
+  <gazebo reference="base_link">
+      <static>true</static>
+      <turnGravityOff>false</turnGravityOff>
+  </gazebo>
 </robot>

Commit message: few fixes for gazebo issue

File: urdf/scara_52900.urdf.xacro (robot description, xacro)
@@ -28,4 +28,8 @@
       <color rgba="1 1 0 1"/>
   </material>
+  <!-- Used for fixing robot to Gazebo 'base_link' -->
+  <link name="world">
+      <origin xyz="0 0 0"/>
+  </link>
   <link name="base_link">
     <visual>
@@ -43,10 +47,8 @@
     <inertial>
     	<mass value="4" />
-      <inertia ixx="1e-3" ixy="0.0" ixz="0.0" iyy="1e-3" iyz="0.0" izz="1e-3"/>
+         <inertia ixx="0.4" ixy="0.0" ixz="0.0" iyy="0.4" iyz="0.0" izz="0.2"/>
       <origin xyz="0 0 0" rpy="0 0 0" />
   	</inertial>
   </link>
-  <!-- Used for fixing robot to Gazebo 'base_link' -->
-  <link name="world"/>
   <joint name="fixed" type="fixed">
     <parent link="world"/>

Commit message: some default PIDs, added rosserial_arduino as dependency

File: urdf/scara_52900.urdf.xacro (robot description, xacro)
@@ -54,5 +54,5 @@
     <parent link="world"/>
     <child link="base_link"/>
-    <origin xyz="0 0 0"/>
+    <origin xyz="0 0 -.93"/>
   </joint>
   <link name="scapula">
@@ -91,5 +91,5 @@
     </actuator>
     <joint name="waist">
-      <hardwareInterface>PositionJointInterface</hardwareInterface>
+      <hardwareInterface>hardware_interface/PositionJointInterface</hardwareInterface>
     </joint>
   </transmission>
@@ -126,5 +126,5 @@
     </actuator>
     <joint name="shoulder">
-      <hardwareInterface>PositionJointInterface</hardwareInterface>
+      <hardwareInterface>hardware_interface/PositionJointInterface</hardwareInterface>
     </joint>
   </transmission>
@@ -161,5 +161,5 @@
     </actuator>
     <joint name="elbow">
-      <hardwareInterface>PositionJointInterface</hardwareInterface>
+      <hardwareInterface>hardware_interface/PositionJointInterface</hardwareInterface>
     </joint>
   </transmission>
@@ -196,5 +196,5 @@
     </actuator>
     <joint name="wrist">
-      <hardwareInterface>PositionJointInterface</hardwareInterface>
+      <hardwareInterface>hardware_interface/PositionJointInterface</hardwareInterface>
     </joint>
   </transmission>

Commit message: add pdf doc from manufacturer, fix z index of base link which corrected gazebo presentation but presented robot below ground level in moveit

File: urdf/scara_52900.urdf.xacro (robot description, xacro)
@@ -54,5 +54,5 @@
     <parent link="world"/>
     <child link="base_link"/>
-    <origin xyz="0 0 -.93"/>
+    <origin xyz="0 0 0"/>
   </joint>
   <link name="scapula">
